Commit message: Added ros control and fixed recon_car_polygon.urdf axes bug

File: bringup/models/reconCarPolygon.urdf (robot description, URDF)
Before this commit: robot recon_car_polygon, 5 links, 4 joints
Links:
- link chassis: geometry collision box size=0.8 0.4 0.2; visual box size=0.8 0.4 0.2
Joints:
- joint chassis_to_frontWheel: origin xyz=0 0.35 -0.15 rpy=0 0 0 -> xyz=0.35 0 -0.15 rpy=0 0 0
- joint chassis_to_leftWheel: axis 1 0 0 -> 0 1 0; origin xyz=-0.22 -0.2 -0.15 rpy=0 0 0 -> xyz=0 0.22 -0.15 rpy=0 0 0
- joint chassis_to_rightWheel: axis 1 0 0 -> 0 1 0; origin xyz=0.22 -0.2 -0.15 rpy=0 0 0 -> xyz=0 -0.22 -0.15 rpy=0 0 0
- joint front_sensor_to_chassis: origin xyz=0 0.4125 0.125 rpy=0 0 1.5707 -> xyz=0.4125 0 0.125 rpy=0 0 0

Commit message: Added slam_toolbox mapping and added rviz into launch file

File: bringup/models/reconCarPolygon.urdf (robot description, URDF)
Before this commit: robot recon_car_polygon, 5 links, 4 joints
Links:
- added link backWheel, mass 0.5; collision sphere radius=0.1; visual sphere radius=0.1
Joints:
- added joint chassis_to_backWheel: type fixed, parent chassis, child backWheel, origin xyz=-0.35 0 -0.15 rpy=0 0 0
- joint chassis_to_leftWheel: origin xyz=0 0.22 -0.15 rpy=0 0 0 -> xyz=0.0 0.22 -0.15 rpy=0 0 0
- joint chassis_to_rightWheel: origin xyz=0 -0.22 -0.15 rpy=0 0 0 -> xyz=0.0 -0.22 -0.15 rpy=0 0 0
