Commit message: Added camera link and topic

File: bringup/models/reconCarPolygon.urdf (robot description, URDF)
Before this commit: robot recon_car_polygon, 6 links, 5 joints
Links:
- added link camera, mass 0.05; collision box size=0.025 0.025 0.01; visual box size=0.025 0.025 0.01
- added link camera_optical
Joints:
- added joint camera_optical_to_camera: type fixed, parent camera, child camera_optical, origin xyz=0.0 0.0 0.0 rpy=-1.5707963268 0.0 -1.5707963268
- added joint camera_to_chassis: type fixed, parent chassis, child camera, origin xyz=0.42 0 0.04 rpy=0 0 0
