Commit message: changed params to match physical robot

File: bringup/models/reconCarMesh.urdf (robot description, URDF)
Before this commit: robot recon_car_polygon, 8 links, 7 joints
Links:
- removed link frontWheel
- link backWheel: geometry collision sphere radius=0.04; visual sphere radius=0.1
- link chassis: geometry collision box size=0.254 0.33 0.102; visual box size=0.254 0.33 0.102
- link leftWheel: geometry collision cylinder length=0.053 radius=0.0559; visual cylinder length=0.053 radius=0.0559
- link rightWheel: geometry collision cylinder length=0.053 radius=0.0559; visual cylinder length=0.053 radius=0.0559
Joints:
- removed joint chassis_to_frontWheel
- joint camera_to_chassis: origin xyz=0.42 0 0.04 rpy=0 0 0 -> xyz=0.122 0 0.0635 rpy=0 0 0
- joint chassis_to_backWheel: origin xyz=-0.35 0 -0.15 rpy=0 0 0 -> xyz=-0.076 0 -0.040 rpy=0 0 0
- joint chassis_to_leftWheel: origin xyz=0.0 0.22 -0.15 rpy=0 0 0 -> xyz=0.076 0.132 -0.043 rpy=0 0 0
- joint chassis_to_rightWheel: origin xyz=0.0 -0.22 -0.15 rpy=0 0 0 -> xyz=0.076 -0.132 -0.043 rpy=0 0 0
- joint front_sensor_to_chassis: origin xyz=0.4125 0 0.125 rpy=0 0 0 -> xyz=-0.0826 0 0.1143 rpy=0 0 0
